Commit message: fix arm to above plate and add end effector manipulation to target position

File: resource/urdf/stretch/stretch.urdf (robot description, URDF)
Before this commit: robot stretch, 25 links, 24 joints
Joints:
- joint joint_lift: origin xyz=-0.037385 0.1666 0 rpy=-1.5708 1.5708 0 -> xyz=-0.037385 0.55 0 rpy=-1.5708 1.5708 0
